File: hackpad.kicad_pcb (KiCad board)
At the start: 2 copper layers, 9 parts, among them SW1 SW_Push, SW2 SW_Push, SW3 SW_Push, SW4 SW_Push, U1 XIAO-RP2040-DIP

Commit message: finished up pcb, organized files, moving onto CAD
Parts:
- moved SW4 64.3 mm to (145.4, 97.3)
- moved D2 61.8 mm to (104.8, 114.3), turned to 180 degrees
- moved D1 61.3 mm to (85.1, 114.3), turned to 180 degrees
- moved D3 51.8 mm to (124.5, 114.3), turned to 180 degrees
- moved D4 31.6 mm to (143.5, 114.3), turned to 180 degrees
- moved SW1 24.7 mm to (88.3, 97.3)
- moved SW3 22.8 mm to (126.4, 97.3)
- moved U1 19.0 mm to (113.8, 81.4)
- moved SW2 9.69 mm to (107.3, 97.3)
Routing:
- net GND: track 0.00 -> 267.7 mm
- net +5V: track 0.00 -> 117.7 mm
- net Net-(U1-GPIO1/RX): track 0.00 -> 44.8 mm
- net Net-(D1-DIN): track 0.00 -> 42.8 mm
- net Net-(U1-GPIO2/SCK): track 0.00 -> 29.3 mm
- net Net-(U1-GPIO3/MOSI): track 0.00 -> 25.7 mm
- net Net-(U1-GPIO4/MISO): track 0.00 -> 17.7 mm
- net Net-(D1-DOUT): track 0.00 -> 16.9 mm
- net Net-(D2-DOUT): track 0.00 -> 16.9 mm
- net Net-(D3-DOUT): track 0.00 -> 16.3 mm
Other:
- board outline added: 76.2 x 45.7 mm
- board text added: "andy sin's hackpad BLEHHH"
- board text added: "xiao here!!!!"
